Commit message: update for macro

File: arm_description/urdf/fotokite_7dof.xacro (robot description, xacro)
@@ -7,15 +7,9 @@
   </gazebo>
   <!-- Geometrical properties -->
-  <xacro:property name="link_side"      value="0.02"/>
-  <xacro:property name="joint_radius"   value="0.018"/>
-  <xacro:property name="joint_length"   value="0.025"/>
-  <xacro:property name="toe_length"     value="0.03"/>
-  <xacro:property name="foot_length"    value="0.04"/>
-  <xacro:property name="knee_length"    value="0.04"/>
-  <xacro:property name="lap_length"     value="0.04"/>
-  <xacro:property name="hip_length"     value="0.04"/>
-  <xacro:property name="arm_length"     value="0.04"/>
-  <xacro:property name="hand_length"    value="0.04"/>
-  <xacro:property name="finger_length"  value="0.04"/>
+  <xacro:property name="link_side"          value="0.02"/>
+  <xacro:property name="joint_radius"       value="0.018"/>
+  <xacro:property name="joint_length"       value="0.025"/>
+  <xacro:property name="shoulder_length"    value="0.04"/>
+  <xacro:property name="wrist_length"       value="0.04"/>
   <!-- Materials -->
   <material name="orange">
@@ -128,20 +122,22 @@
   </xacro:macro>
   <!-- Uncomment for RViz with fake joints -->
-  <!-- World frame (for Gazebo) -->
-  <!--link name="world"/-->
+  <!-- Uncomment for Gazebo -->
+  <link name="base_link"/>
   <!-- Uncomment for RViz with fake joints -->
+  <!-- Uncomment for Gazebo -->
   <!-- Arm fixed to world frame  -->
-  <!--joint name="world_foot_joint" type="fixed">
-    <parent link="world"/>
-    <child link="toe"/>
-  </joint-->
+  <joint name="shoulder_joint" type="fixed">
+      <origin xyz="-0.25 0.10 0.275" rpy="0 0 0"/>
+      <parent link="base_link"/>
+      <child link="shoulder_yaw"/>
+  </joint>
   <!-- Joints Chain -->
-  <xacro:arm_joint parent="toe"     child="foot"    axis="0 0 1" dist="${toe_length}"   joint_type="revolute"   lower="${-PI}"      upper="${PI}"   />
-  <xacro:arm_joint parent="foot"    child="knee"    axis="1 0 0" dist="${foot_length}"  joint_type="revolute"   lower="${-PI}"      upper="${PI}"   />
-  <xacro:arm_joint parent="knee"    child="lap"     axis="0 1 0" dist="${knee_length}"  joint_type="revolute"   lower="${-PI}"      upper="${PI}"   />
-  <xacro:arm_joint parent="lap"     child="hip"     axis="0 0 1" dist="${lap_length}"   joint_type="prismatic"  lower="0"           upper="2"       />
-  <xacro:arm_joint parent="hip"     child="arm"     axis="0 0 1" dist="${hip_length}"   joint_type="revolute"   lower="${-PI}"      upper="${PI}"   />
-  <xacro:arm_joint parent="arm"     child="hand"    axis="0 1 0" dist="${arm_length}"   joint_type="revolute"   lower="${-PI}"      upper="${PI}"   />
-  <xacro:arm_joint parent="hand"    child="finger"  axis="1 0 0" dist="${hand_length}"  joint_type="revolute"   lower="${-PI}"      upper="${PI}"   />
+  <xacro:arm_joint parent="shoulder_yaw"      child="shoulder_roll"   axis="0 0 1" dist="${shoulder_length}"    joint_type="revolute"   lower="${-PI}"      upper="${PI}"   />
+  <xacro:arm_joint parent="shoulder_roll"     child="shoulder_pitch"  axis="1 0 0" dist="${shoulder_length}"    joint_type="revolute"   lower="${-PI/2}"    upper="${PI/2}" />
+  <xacro:arm_joint parent="shoulder_pitch"    child="arm_length"      axis="0 1 0" dist="${shoulder_length}"    joint_type="revolute"   lower="${-PI/2}"    upper="${PI/2}" />
+  <xacro:arm_joint parent="arm_length"        child="wrist_yaw"       axis="0 0 1" dist="${shoulder_length}"    joint_type="prismatic"  lower="0"           upper="2"       />
+  <xacro:arm_joint parent="wrist_yaw"         child="wrist_roll"      axis="0 0 1" dist="${wrist_length}"       joint_type="revolute"   lower="${-PI}"      upper="${PI}"   />
+  <xacro:arm_joint parent="wrist_roll"        child="wrist_pitch"     axis="0 1 0" dist="${wrist_length}"       joint_type="revolute"   lower="${-PI}"      upper="${PI}"   />
+  <xacro:arm_joint parent="wrist_pitch"       child="finger"          axis="1 0 0" dist="${wrist_length}"       joint_type="revolute"   lower="${-PI}"      upper="${PI}"   />
   <!-- End effector -->
   <!--link name="finger">
@@ -159,5 +155,5 @@
         <origin xyz="0 0 0" rpy="0 0 0" />
         <geometry>
-          <mesh filename="package://arm_description/urdf/ardrone.dae"/>
+          <mesh filename="package://arm_description/meshes/ardrone.dae"/>
         </geometry>
       </visual>

File: arm_description/urdf/fotokite_7dof_two_modules.xacro (robot description, xacro)
@@ -167,5 +167,5 @@
         <origin xyz="0 0 0" rpy="0 0 0" />
         <geometry>
-          <mesh filename="package://arm_description/urdf/ardrone.dae"/>
+          <mesh filename="package://arm_description/meshes/ardrone.dae"/>
         </geometry>
       </visual>
